File: pcb/espxpansion.kicad_pcb (KiCad board)
At the start: 2 copper layers, 32 x 25.5 mm, 13 parts, among them J2 Conn_01x02_Pin, U1 ESP32-C6-MINI-1

Commit message: stuffs meow
Parts:
- added R5: 10k, Resistor_SMD:R_0402_1005Metric, F.Cu at (95.5, 98.5)
Connections:
- U1 pad 22: unconnected-(U1-IO8-Pad22) -> Net-(U1-IO8)
Routing:
- net Net-(U1-IO8): track 0.00 -> 5.49 mm, vias 0 -> 2
Other:
- board text added: "ESP"
- board text added: "for Hackxpansion"

Commit message: fixes
Parts:
- removed C1: 100nF, Capacitor_SMD:C_0402_1005Metric
- J2: footprint Connector_PinHeader_2.54mm:PinHeader_1x02_P2.54mm_Vertical -> Connector_PinHeader_2.54mm:PinHeader_1x04_P2.54mm_Vertical
- moved J2 0.52 mm to (88.6, 92.0)
Connections:
- J2 pad 1: /ESP_TX -> +3V3
- J2 pad 2: /ESP_RX -> /ESP_TX
Routing:
- net +3V3: track 76.5 -> 85.1 mm, vias 0 -> 1
- net /ESP_RX: track 36.0 -> 32.8 mm
- net /ESP_TX: track 32.5 -> 34.0 mm
- net GND: track 7.00 -> 5.96 mm, vias 18 -> 19
