File: pcb/espxpansion.kicad_sch (KiCad schematic)
At the start: 11 parts, among them J2 Conn_01x02_Pin, SW1 BOOT, SW2 RESET, U1 ESP32-C6-MINI-1

Commit message: stuffs meow
Parts:
- added R5: 10k, Resistor_SMD:R_0402_1005Metric, symbol Device:R
- C1: LCSC Part # (none) -> C60474
- C2: LCSC Part # (none) -> C76991
- R1: LCSC Part # (none) -> C140197
- R2: LCSC Part # (none) -> C2906867
- R3, R4: LCSC Part # (none) -> C2906861
- SW1, SW2: LCSC Part # (none) -> C720477
- U1: LCSC Part # (none) -> C5736265
Connections:
- net +3V3: now also R5.1
- net at U1.22 (IO8): now also R5.2
- no-connect marks 23 -> 22

Commit message: fixes
Parts:
- removed C1: 100nF, Capacitor_SMD:C_0402_1005Metric, symbol Device:C
- J2: footprint Connector_PinHeader_2.54mm:PinHeader_1x02_P2.54mm_Vertical -> Connector_PinHeader_2.54mm:PinHeader_1x04_P2.54mm_Vertical; symbol Connector:Conn_01x02_Pin -> Connector:Conn_01x04_Pin
Connections:
- net +3V3: now also J2.1 (Pin_1)
- net ESP_RX: now also J2.3 (Pin_3); no longer J2.2 (Pin_2)
- net ESP_TX: now also J2.2 (Pin_2); no longer J2.1 (Pin_1)
- net GND: now also J2.4 (Pin_4)
Other:
- moved on the sheet: C2
